Commit message: update 260224

File: src/kaair_description/urdf/head/head.ros2_control.xacro (robot description, xacro)
@@ -1,19 +1,27 @@
 <?xml version="1.0"?>
 <robot xmlns:xacro="http://www.ros.org/wiki/xacro">
-  <xacro:macro name="head_ros2_control" params="name usb_port baud_rate">
+  <xacro:macro name="head_ros2_control" params="name spec use_fake_hardware:=false">
     <ros2_control name="${name}" type="system">
       <hardware>
-        <plugin>kaair_driver/HeadHwInterface</plugin>
-        <param name="usb_port">${usb_port}</param>
-        <param name="baud_rate">${baud_rate}</param>
+        <xacro:if value="${use_fake_hardware}">
+          <plugin>mock_components/GenericSystem</plugin>
+          <param name="calculate_dynamics">true</param>
+        </xacro:if>
+        <xacro:unless value="${use_fake_hardware}">
+          <plugin>kaair_driver/HeadHwInterface</plugin>
+          <param name="usb_port">${spec['usb_port']}</param>
+          <param name="baud_rate">${spec['baud_rate']}</param>
+        </xacro:unless>
       </hardware>
       <joint name="head_joint1">
         <command_interface name="position"/>
-        <state_interface name="position"/>
+        <state_interface name="position">
+          <param name="initial_value">0.0</param> </state_interface>
         <param name="id">1</param>
       </joint>
       <joint name="head_joint2">
         <command_interface name="position"/>
-        <state_interface name="position"/>
+        <state_interface name="position">
+          <param name="initial_value">0.0</param> </state_interface>
        <param name="id">2</param>
       </joint>

File: src/kaair_description/urdf/lift/lift.urdf.xacro (robot description, xacro)
@@ -3,6 +3,4 @@
   <xacro:property name="m_to_mm" value="0.001 0.001 0.001"/>
   <xacro:property name="mesh_path" value="package://kaair_description/meshes/"/>
-  <xacro:arg name="lift_lower_limit" default="0.100"/>
-  <xacro:arg name="lift_upper_limit" default="0.600"/>
   <xacro:macro name="lift_module" params="min_h max_h">
     <link name="lift_base_link">
@@ -46,7 +44,5 @@
       <axis xyz="0.0 0.0 1.0"/>
       <limit
-        upper="$(arg lift_upper_limit)"
-        lower="$(arg lift_lower_limit)"
-        effort="700"
+        upper="${max_h}"  lower="${min_h}"  effort="700"
         velocity="0.34"/>
     </joint>

File: src/kaair_description/urdf/robot.urdf.xacro (robot description, xacro)
@@ -2,11 +2,18 @@
 <robot name="kaair" xmlns:xacro="http://www.ros.org/wiki/xacro">
   <xacro:arg name="mode" default="robot"/>
-  <xacro:arg name="lift_lower_limit" default="0.100"/>
-  <xacro:arg name="lift_upper_limit" default="0.700"/>
+  <xacro:arg name="hw_spec_file" default="$(find kaair_bringup)/config/robots/kaair_specs_01.yaml"/>
+  <xacro:arg name="use_fake_hardware" default="false"/>
+  <xacro:property name="hw_specs" value="${xacro.load_yaml('$(arg hw_spec_file)')}"/>
   <xacro:if value="${'$(arg mode)' == 'robot' or '$(arg mode)' == 'lift'}">
     <xacro:include filename="$(find kaair_description)/urdf/lift/lift.urdf.xacro"/>
+    <xacro:include filename="$(find kaair_description)/urdf/lift/lift.ros2_control.xacro"/>
     <xacro:lift_module
-      min_h="$(arg lift_lower_limit)"
-      max_h="$(arg lift_upper_limit)"
+      min_h="${hw_specs['lift']['min_h']}"
+      max_h="${hw_specs['lift']['max_h']}"
+    />
+    <xacro:lift_ros2_control
+      name="LiftHardware"
+      spec="${hw_specs['lift']}"
+      use_fake_hardware="$(arg use_fake_hardware)"
     />
   </xacro:if>
@@ -16,6 +23,6 @@
     <xacro:head_ros2_control
       name="HeadHardware"
-      usb_port="/dev/ttyHead"
-      baud_rate="57600"
+      spec="${hw_specs['head']}"
+      use_fake_hardware="$(arg use_fake_hardware)"
     />
     <xacro:if value="${'$(arg mode)' == 'robot'}">
@@ -31,4 +38,8 @@
       <link name="arm_base"/>
     </xacro:unless>
+    <xacro:property name="arm_hw_plugin" value="uf_robot_hardware/UFRobotSystemHardware"/>
+    <xacro:if value="$(arg use_fake_hardware)">
+      <xacro:property name="arm_hw_plugin" value="uf_robot_hardware/UFRobotFakeSystemHardware"/>
+    </xacro:if>
     <xacro:include filename="$(find xarm_description)/urdf/xarm_device_macro.xacro"/>
     <xacro:xarm_device
@@ -36,8 +47,9 @@
       hw_ns="xarm"
       dof="7"
-      add_gripper="false"
       attach_to="arm_base"
-      attach_xyz="0 0 0"
-      attach_rpy="0 0 0"
+      effort_control="true"
+      velocity_control="true"
+      robot_ip="${hw_specs['arm']['robot_ip']}"
+      ros2_control_plugin="${arm_hw_plugin}"
     />
   </xacro:if>
