Commit message: test moveit example

File: src/kaair_description/urdf/head/head.urdf.xacro (robot description, xacro)
@@ -67,5 +67,5 @@
     </collision>
   </link>
-  <link name="femto_base_link">
+  <link name="head_camera_mount">
   </link>
   <joint name="head_fix_joint" type="fixed">
@@ -83,5 +83,5 @@
       upper="1.58"
       effort="30"
-      velocity="3.14" />
+      velocity="1.2" />
   </joint>
   <joint name="head_joint2" type="revolute">
@@ -94,10 +94,10 @@
       upper="1.58"
       effort="30"
-      velocity="3.14" />
+      velocity="1.2" />
   </joint>
   <joint name="pantilt_femto_frame_joint" type="fixed">
     <origin xyz="0.0 0.0 0.055" rpy="0 0 0"/>
     <parent link="head_link3"/>
-    <child link="femto_base_link"/>
+    <child link="head_camera_mount"/>
   </joint>
 </robot>

File: src/kaair_description/urdf/robot.urdf.xacro (robot description, xacro)
@@ -21,4 +21,5 @@
     <xacro:include filename="$(find kaair_description)/urdf/head/head.urdf.xacro"/>
     <xacro:include filename="$(find kaair_description)/urdf/head/head.ros2_control.xacro"/>
+    <xacro:include filename="$(find orbbec_description)/urdf/femto_bolt.urdf.xacro"/>
     <xacro:head_ros2_control
       name="HeadHardware"
@@ -26,4 +27,7 @@
       use_fake_hardware="$(arg use_fake_hardware)"
     />
+  <xacro:femto_bolt prefix="femto" parent="head_camera_mount">
+    <origin xyz="0 0 0" rpy="0 0 0" />
+  </xacro:femto_bolt>
     <xacro:if value="${'$(arg mode)' == 'robot'}">
       <joint name="lift_to_head_fix_joint" type="fixed">
