Commit message: Update Lift UDRF and processing lift hw_interface

File: src/kaair_description/urdf/lift/lift.urdf.xacro (robot description, xacro)
@@ -1,9 +1,11 @@
 <?xml version="1.0" ?>
 <robot name="lift" xmlns:xacro="http://www.ros.org/wiki/xacro">
+  <xacro:property name="m_to_mm" value="0.001 0.001 0.001"/>
+  <xacro:property name="mesh_path" value="package://kaair_description/meshes/"/>
   <link name="lift_base_link">
     <!-- visual -->
     <visual>
       <geometry>
-        <mesh filename="package://keti_assist_ai_robot_description/meshes/lift/visual/lift_base.stl"/>
+        <mesh filename="${mesh_path}lift/visual/lift_base.stl" scale="${m_to_mm}"/>
       </geometry>
       <origin xyz="0 0 0" rpy="0 0 0"/>
@@ -12,5 +14,5 @@
     <collision>
       <geometry>
-        <mesh filename="package://keti_assist_ai_robot_description/meshes/lift/visual/lift_base.stl"/>
+        <mesh filename="${mesh_path}lift/visual/lift_base.stl" scale="${m_to_mm}"/>
       </geometry>
       <origin xyz="0 0 0" rpy="0 0 0"/>
@@ -21,5 +23,5 @@
     <visual>
       <geometry>
-        <mesh filename="package://keti_assist_ai_robot_description/meshes/lift/visual/lift_link.stl"/>
+        <mesh filename="${mesh_path}lift/visual/lift_link.stl" scale="${m_to_mm}"/>
       </geometry>
       <origin xyz="0 0 0" rpy="0 0 0"/>
@@ -28,5 +30,5 @@
     <collision>
       <geometry>
-        <mesh filename="package://keti_assist_ai_robot_description/meshes/lift/visual/lift_link.stl"/>
+        <mesh filename="${mesh_path}lift/visual/lift_link.stl" scale="${m_to_mm}"/>
       </geometry>
       <origin xyz="0 0 0" rpy="0 0 0"/>

Commit message: urdf optimizing

File: src/kaair_description/urdf/lift/lift.urdf.xacro (robot description, xacro)
@@ -3,42 +3,54 @@
   <xacro:property name="m_to_mm" value="0.001 0.001 0.001"/>
   <xacro:property name="mesh_path" value="package://kaair_description/meshes/"/>
-  <link name="lift_base_link">
-    <!-- visual -->
-    <visual>
-      <geometry>
-        <mesh filename="${mesh_path}lift/visual/lift_base.stl" scale="${m_to_mm}"/>
-      </geometry>
-      <origin xyz="0 0 0" rpy="0 0 0"/>
-    </visual>
-    <!-- collision -->
-    <collision>
-      <geometry>
-        <mesh filename="${mesh_path}lift/visual/lift_base.stl" scale="${m_to_mm}"/>
-      </geometry>
-      <origin xyz="0 0 0" rpy="0 0 0"/>
-    </collision>
-  </link>
-  <link name="lift_link">
-    <!-- visual -->
-    <visual>
-      <geometry>
-        <mesh filename="${mesh_path}lift/visual/lift_link.stl" scale="${m_to_mm}"/>
-      </geometry>
-      <origin xyz="0 0 0" rpy="0 0 0"/>
-    </visual>
-    <!-- collision -->
-    <collision>
-      <geometry>
-        <mesh filename="${mesh_path}lift/visual/lift_link.stl" scale="${m_to_mm}"/>
-      </geometry>
-      <origin xyz="0 0 0" rpy="0 0 0"/>
-    </collision>
-  </link>
-  <joint name="lift_joint" type="prismatic">
-    <origin xyz="0.0 0.0 0.0" rpy="0 0 0"/>
-    <parent link="lift_base_link"/>
-    <child link="lift_link"/>
-    <axis xyz="0.0 0.0 1.0"/>
-    <limit upper="0.8" lower="0.0" effort="100" velocity="100"/>
-  </joint>
+  <xacro:arg name="lift_lower_limit" default="0.100"/>
+  <xacro:arg name="lift_upper_limit" default="0.600"/>
+  <xacro:macro name="lift_module" params="min_h max_h">
+    <link name="lift_base_link">
+      <!-- visual -->
+      <visual>
+        <geometry>
+          <mesh filename="${mesh_path}lift/visual/lift_base.stl" scale="${m_to_mm}"/>
+        </geometry>
+        <origin xyz="0 0 0" rpy="0 0 0"/>
+      </visual>
+      <!-- collision -->
+      <collision>
+        <geometry>
+          <mesh filename="${mesh_path}lift/collision/lift_base.stl" scale="${m_to_mm}"/>
+        </geometry>
+        <origin xyz="0 0 0" rpy="0 0 0"/>
+      </collision>
+    </link>
+    <link name="lift_link">
+      <!-- visual -->
+      <visual>
+        <geometry>
+          <mesh filename="${mesh_path}lift/visual/lift_link.stl" scale="${m_to_mm}"/>
+        </geometry>
+        <origin xyz="0 0 0" rpy="0 0 0"/>
+      </visual>
+      <!-- collision -->
+      <collision>
+        <geometry>
+          <mesh filename="${mesh_path}lift/collision/lift_link.stl" scale="${m_to_mm}"/>
+        </geometry>
+        <origin xyz="0 0 0" rpy="0 0 0"/>
+      </collision>
+    </link>
+    <joint name="lift_joint" type="prismatic">
+      <origin xyz="0.0 0.0 0.0" rpy="0 0 0"/>
+      <parent link="lift_base_link"/>
+      <child link="lift_link"/>
+      <axis xyz="0.0 0.0 1.0"/>
+      <limit
+        upper="$(arg lift_upper_limit)"
+        lower="$(arg lift_lower_limit)"
+        effort="100"
+        velocity="100"/>
+    </joint>
+  </xacro:macro>
+  <xacro:lift_module
+    min_h="$(arg lift_lower_limit)"
+    max_h="$(arg lift_upper_limit)"
+  />
 </robot>

Commit message: Update Head hw

File: src/kaair_description/urdf/lift/lift.urdf.xacro (robot description, xacro)
@@ -38,4 +38,6 @@
       </collision>
     </link>
+    <link name="arm_base">
+    </link>
     <joint name="lift_joint" type="prismatic">
       <origin xyz="0.0 0.0 0.0" rpy="0 0 0"/>
@@ -46,11 +48,12 @@
         upper="$(arg lift_upper_limit)"
         lower="$(arg lift_lower_limit)"
-        effort="100"
-        velocity="100"/>
+        effort="700"
+        velocity="0.34"/>
+    </joint>
+    <joint name="lift_to_arm_fix_joint" type="fixed">
+      <origin xyz="0.2415 0.0 0.0" rpy="0 0 0"/>
+      <parent link="lift_link"/>
+      <child link="arm_base"/>
     </joint>
   </xacro:macro>
-  <xacro:lift_module
-    min_h="$(arg lift_lower_limit)"
-    max_h="$(arg lift_upper_limit)"
-  />
 </robot>

File: src/kaair_description/urdf/robot.urdf.xacro (robot description, xacro)
@@ -1,21 +1,44 @@
 <?xml version="1.0" ?>
 <robot name="kaair" xmlns:xacro="http://www.ros.org/wiki/xacro">
+  <xacro:arg name="mode" default="robot"/>
   <xacro:arg name="lift_lower_limit" default="0.100"/>
-  <xacro:arg name="lift_upper_limit" default="0.600"/>
-  <xacro:include filename="$(find kaair_description)/urdf/lift/lift.urdf.xacro"/>
-  <xacro:lift_module
-    min_h="$(arg lift_lower_limit)"
-    max_h="$(arg lift_upper_limit)"
-  />
-  <xacro:include filename="$(find kaair_description)/urdf/head/head.urdf.xacro"/>
-  <!-- <joint name="lift_to_arm_fix_joint" type="fixed">
-    <origin xyz="0.2415 0.0 0.0" rpy="0 0 0"/>
-    <parent link="lift_link"/>
-    <child link="world"/>
-  </joint> -->
-  <joint name="lift_to_head_fix_joint" type="fixed">
-    <origin xyz="0.0 0.0 0.859" rpy="0 0 0"/>
-    <parent link="lift_base_link"/>
-    <child link="head_base"/>
-  </joint>
+  <xacro:arg name="lift_upper_limit" default="0.700"/>
+  <xacro:if value="${'$(arg mode)' == 'robot' or '$(arg mode)' == 'lift'}">
+    <xacro:include filename="$(find kaair_description)/urdf/lift/lift.urdf.xacro"/>
+    <xacro:lift_module
+      min_h="$(arg lift_lower_limit)"
+      max_h="$(arg lift_upper_limit)"
+    />
+  </xacro:if>
+  <xacro:if value="${'$(arg mode)' == 'robot' or '$(arg mode)' == 'head'}">
+    <xacro:include filename="$(find kaair_description)/urdf/head/head.urdf.xacro"/>
+    <xacro:include filename="$(find kaair_description)/urdf/head/head.ros2_control.xacro"/>
+    <xacro:head_ros2_control
+      name="HeadHardware"
+      usb_port="/dev/ttyHead"
+      baud_rate="57600"
+    />
+    <xacro:if value="${'$(arg mode)' == 'robot'}">
+      <joint name="lift_to_head_fix_joint" type="fixed">
+        <origin xyz="0.0 0.0 0.859" rpy="0 0 0"/>
+        <parent link="lift_base_link"/>
+        <child link="head_base"/>
+      </joint>
+    </xacro:if>
+  </xacro:if>
+  <xacro:if value="${'$(arg mode)' == 'robot' or '$(arg mode)' == 'arm'}">
+    <xacro:unless value="${'$(arg mode)' == 'robot'}">
+      <link name="arm_base"/>
+    </xacro:unless>
+    <xacro:include filename="$(find xarm_description)/urdf/xarm_device_macro.xacro"/>
+    <xacro:xarm_device
+      prefix=""
+      hw_ns="xarm"
+      dof="7"
+      add_gripper="false"
+      attach_to="arm_base"
+      attach_xyz="0 0 0"
+      attach_rpy="0 0 0"
+    />
+  </xacro:if>
 </robot>

Commit message: moveit real tested

File: src/kaair_description/urdf/lift/lift.urdf.xacro (robot description, xacro)
@@ -11,4 +11,5 @@
         </geometry>
         <origin xyz="0 0 0" rpy="0 0 0"/>
+        <material name="gray"/>
       </visual>
       <!-- collision -->
@@ -27,4 +28,5 @@
         </geometry>
         <origin xyz="0 0 0" rpy="0 0 0"/>
+        <material name="light_gray"/>
       </visual>
       <!-- collision -->

File: src/kaair_description/urdf/robot.urdf.xacro (robot description, xacro)
@@ -1,4 +1,19 @@
 <?xml version="1.0" ?>
 <robot name="kaair" xmlns:xacro="http://www.ros.org/wiki/xacro">
+  <material name="black">
+    <color rgba="0.0 0.0 0.0 1.0"/>
+  </material>
+  <material name="white">
+    <color rgba="1.0 1.0 1.0 1.0"/>
+  </material>
+  <material name="gray">
+    <color rgba="0.5 0.5 0.5 1.0"/>
+  </material>
+  <material name="dark_gray">
+    <color rgba="0.2 0.2 0.2 1.0"/>
+  </material>
+  <material name="light_gray">
+    <color rgba="0.8 0.8 0.8 1.0"/>
+  </material>
   <xacro:arg name="mode" default="robot"/>
   <xacro:arg name="hw_spec_file" default="$(find kaair_bringup)/config/robots/kaair_specs_01.yaml"/>

File: src/kaair_description/urdf/tool/tool.urdf.xacro (robot description, xacro)
@@ -10,4 +10,5 @@
         </geometry>
         <origin xyz="0 0 0" rpy="0 0 0"/>
+        <material name="gray"/>
       </visual>
       <!-- collision -->
@@ -26,4 +27,5 @@
         </geometry>
         <origin xyz="0 0 0" rpy="0 0 0"/>
+        <material name="light_gray"/>
       </visual>
       <!-- collision -->
@@ -42,4 +44,5 @@
         </geometry>
         <origin xyz="0 0 0" rpy="0 0 0"/>
+        <material name="black"/>
       </visual>
       <!-- collision -->
@@ -58,4 +61,5 @@
         </geometry>
         <origin xyz="0 0 0" rpy="0 0 0"/>
+        <material name="dark_gray"/>
       </visual>
       <!-- collision -->
@@ -74,4 +78,5 @@
         </geometry>
         <origin xyz="0 0 0" rpy="0 0 0"/>
+        <material name="dark_gray"/>
       </visual>
       <!-- collision -->

File: src/kaair_moveit_config/config/kaair.ros2_control.xacro (robot description, xacro)
@@ -64,11 +64,4 @@
                 <state_interface name="velocity"/>
             </joint>
-            <joint name="virtual_gripper_joint">
-                <command_interface name="position"/>
-                <state_interface name="position">
-                  <param name="initial_value">${initial_positions['virtual_gripper_joint']}</param>
-                </state_interface>
-                <state_interface name="velocity"/>
-            </joint>
         </ros2_control>
     </xacro:macro>
