Commit message: Need to integrate one control manager

File: src/kaair_description/urdf/robot.urdf.xacro (robot description, xacro)
@@ -47,4 +47,5 @@
       hw_ns="xarm"
       dof="7"
+      add_gripper="false"
       attach_to="arm_base"
       effort_control="true"
@@ -54,3 +55,19 @@
     />
   </xacro:if>
+  <xacro:if value="${'$(arg mode)' == 'robot' or '$(arg mode)' == 'tool'}">
+    <xacro:include filename="$(find kaair_description)/urdf/tool/tool.urdf.xacro"/>
+    <xacro:include filename="$(find kaair_description)/urdf/tool/tool_ros2_control.xacro"/>
+    <xacro:if value="${'$(arg mode)' == 'robot'}">
+      <joint name="arm_to_tool_fix_joint" type="fixed">
+        <origin xyz="0.0 0.0 0.0" rpy="0 0 0"/>
+        <parent link="link_eef"/>
+        <child link="hand_base_link"/>
+      </joint>
+    </xacro:if>
+    <xacro:tool_ros2_control
+      name="ToolHardware"
+      spec="${hw_specs['tool']}"
+      use_fake_hardware="$(arg use_fake_hardware)"
+    />
+  </xacro:if>
 </robot>

File: src/kaair_description/urdf/tool/tool_ros2_control.xacro (robot description, xacro)
@@ -1,9 +1,7 @@
 <?xml version="1.0"?>
 <robot xmlns:xacro="http://www.ros.org/wiki/xacro">
-  <xacro:macro name="lift_ros2_control" params="name spec use_fake_hardware:=false">
+  <xacro:macro name="tool_ros2_control" params="name spec use_fake_hardware:=false">
     <ros2_control name="${name}" type="system">
       <hardware>
-        <param name="min_height">${spec['min_h']}</param>
-        <param name="max_height">${spec['max_h']}</param>
         <xacro:if value="${use_fake_hardware}">
           <plugin>mock_components/GenericSystem</plugin>
@@ -11,14 +9,14 @@
         </xacro:if>
         <xacro:unless value="${use_fake_hardware}">
-          <plugin>kaair_driver/LiftHwInterface</plugin>
+          <plugin>kaair_driver/ToolHwInterface</plugin>
           <param name="serial_port">${spec['usb_port']}</param>
           <param name="baud_rate">${spec['baud_rate']}</param>
         </xacro:unless> </hardware>
-      <joint name="lift_joint">
+      <joint name="right_finger_tip_joint">
           <command_interface name="position">
           </command_interface>
           <command_interface name="velocity"/>
           <state_interface name="position">
-            <param name="initial_value">${spec['initial_pose']}</param>
+            <param name="initial_value">0.055</param>
           </state_interface>
           <state_interface name="velocity">

Commit message: mobile description added

File: src/kaair_description/urdf/robot.urdf.xacro (robot description, xacro)
@@ -5,4 +5,7 @@
   <xacro:arg name="use_fake_hardware" default="false"/>
   <xacro:property name="hw_specs" value="${xacro.load_yaml('$(arg hw_spec_file)')}"/>
+  <xacro:if value="${'$(arg mode)' == 'robot' or '$(arg mode)' == 'slamtec'}">
+    <xacro:include filename="$(find kaair_description)/urdf/slamtec/slamtec.urdf.xacro"/>
+  </xacro:if>
   <xacro:if value="${'$(arg mode)' == 'robot' or '$(arg mode)' == 'lift'}">
     <xacro:include filename="$(find kaair_description)/urdf/lift/lift.urdf.xacro"/>
@@ -17,4 +20,11 @@
       use_fake_hardware="$(arg use_fake_hardware)"
     />
+    <xacro:if value="${'$(arg mode)' == 'robot'}">
+      <joint name="lift_to_mobile_joint" type="fixed">
+        <origin xyz="0.0 0.0 0.0" rpy="0 0 0"/>
+        <parent link="robot_base_link"/>
+        <child link="lift_base_link"/>
+      </joint>
+    </xacro:if>
   </xacro:if>
   <xacro:if value="${'$(arg mode)' == 'robot' or '$(arg mode)' == 'head'}">

Commit message: head offeset

File: src/kaair_description/urdf/robot.urdf.xacro (robot description, xacro)
@@ -53,5 +53,5 @@
     />
   <xacro:femto_bolt prefix="femto" parent="head_camera_mount">
-    <origin xyz="0 0 0" rpy="0 0 0" />
+    <origin xyz="0 0 0.01" rpy="0 0 0" />
   </xacro:femto_bolt>
     <xacro:if value="${'$(arg mode)' == 'robot'}">

Commit message: update urdf with realsense

File: src/kaair_description/urdf/robot.urdf.xacro (robot description, xacro)
@@ -99,4 +99,9 @@
       use_fake_hardware="$(arg use_fake_hardware)"
     />
+    <xacro:arg name="use_nominal_extrinsics" default="false"/>
+    <xacro:include filename="$(find realsense2_description)/urdf/_d405.urdf.xacro" />
+    <xacro:sensor_d405 parent="vision_frame_link" use_nominal_extrinsics="$(arg use_nominal_extrinsics)">
+      <origin xyz="0.04428 0 0.02185" rpy="0 -1.5707963267948966 -3.1415926535897931"/>
+    </xacro:sensor_d405>
   </xacro:if>
 </robot>

File: src/kaair_moveit_config/config/kaair.urdf.xacro (robot description, xacro)
@@ -2,7 +2,4 @@
 <robot xmlns:xacro="http://www.ros.org/wiki/xacro" name="kaair">
     <xacro:arg name="initial_positions_file" default="initial_positions.yaml" />
-    <xacro:arg name="use_fake_hardware" default="true" />
-    <xacro:arg name="mode" default="robot" />
-    <xacro:property name="hw_specs" value="${xacro.load_yaml('$(arg hw_spec_file)')}"/>
     <!-- Import kaair urdf file -->
     <xacro:include filename="$(find kaair_description)/urdf/robot.urdf.xacro" />

Commit message: urdf fix

File: src/kaair_description/urdf/robot.urdf.xacro (robot description, xacro)
@@ -89,5 +89,5 @@
     <xacro:if value="${'$(arg mode)' == 'robot'}">
       <joint name="arm_to_tool_fix_joint" type="fixed">
-        <origin xyz="0.0 0.0 0.0" rpy="0 0 0"/>
+        <origin xyz="0.0 0.0 0.0" rpy="0 0 3.1415926535897931"/>
         <parent link="link_eef"/>
         <child link="hand_base_link"/>
@@ -100,4 +100,5 @@
     />
     <xacro:arg name="use_nominal_extrinsics" default="false"/>
+    <xacro:arg name="add_plug" default="true"/>
     <xacro:include filename="$(find realsense2_description)/urdf/_d405.urdf.xacro" />
     <xacro:sensor_d405 parent="vision_frame_link" use_nominal_extrinsics="$(arg use_nominal_extrinsics)">

Commit message: moveit srdf fixing

File: src/kaair_description/urdf/robot.urdf.xacro (robot description, xacro)
@@ -30,9 +30,12 @@
       max_h="${hw_specs['lift']['max_h']}"
     />
-    <xacro:lift_ros2_control
-      name="LiftHardware"
-      spec="${hw_specs['lift']}"
-      use_fake_hardware="$(arg use_fake_hardware)"
-    />
+    <!-- real hw only: fake mode uses kaair_moveit_config/kaair.ros2_control.xacro FakeSystem -->
+    <xacro:unless value="$(arg use_fake_hardware)">
+      <xacro:lift_ros2_control
+        name="LiftHardware"
+        spec="${hw_specs['lift']}"
+        use_fake_hardware="false"
+      />
+    </xacro:unless>
     <xacro:if value="${'$(arg mode)' == 'robot'}">
       <joint name="lift_to_mobile_joint" type="fixed">
@@ -47,9 +50,12 @@
     <xacro:include filename="$(find kaair_description)/urdf/head/head.ros2_control.xacro"/>
     <xacro:include filename="$(find orbbec_description)/urdf/femto_bolt.urdf.xacro"/>
-    <xacro:head_ros2_control
-      name="HeadHardware"
-      spec="${hw_specs['head']}"
-      use_fake_hardware="$(arg use_fake_hardware)"
-    />
+    <!-- real hw only: fake mode uses kaair_moveit_config/kaair.ros2_control.xacro FakeSystem -->
+    <xacro:unless value="$(arg use_fake_hardware)">
+      <xacro:head_ros2_control
+        name="HeadHardware"
+        spec="${hw_specs['head']}"
+        use_fake_hardware="false"
+      />
+    </xacro:unless>
   <xacro:femto_bolt prefix="femto" parent="head_camera_mount">
     <origin xyz="0 0 0.01" rpy="0 0 0" />
@@ -94,9 +100,12 @@
       </joint>
     </xacro:if>
-    <xacro:tool_ros2_control
-      name="ToolHardware"
-      spec="${hw_specs['tool']}"
-      use_fake_hardware="$(arg use_fake_hardware)"
-    />
+    <!-- real hw only: fake mode uses kaair_moveit_config/kaair.ros2_control.xacro FakeSystem -->
+    <xacro:unless value="$(arg use_fake_hardware)">
+      <xacro:tool_ros2_control
+        name="ToolHardware"
+        spec="${hw_specs['tool']}"
+        use_fake_hardware="false"
+      />
+    </xacro:unless>
     <xacro:arg name="use_nominal_extrinsics" default="false"/>
     <xacro:arg name="add_plug" default="true"/>

File: src/kaair_moveit_config/config/kaair.ros2_control.xacro (robot description, xacro)
@@ -1,64 +1,46 @@
 <?xml version="1.0"?>
 <robot xmlns:xacro="http://www.ros.org/wiki/xacro">
+    <!--
+        MoveIt FakeSystem for KAAIR-specific joints only.
+        Arm joints (joint1–joint7) are intentionally excluded here.
+        They are provided by UFRobotFakeSystemHardware inside robot.urdf.xacro
+        when use_fake_hardware=true, so claiming them again would cause a
+        ros2_control ResourceManager conflict.
+        Covered joints:
+          - lift_joint          (LiftHwInterface in real mode)
+          - head_joint1/2       (HeadHwInterface in real mode)
+          - virtual_gripper_joint (ToolHwInterface in real mode)
+    -->
     <xacro:macro name="kaair_ros2_control" params="name initial_positions_file">
         <xacro:property name="initial_positions" value="${load_yaml(initial_positions_file)['initial_positions']}"/>
         <ros2_control name="${name}" type="system">
             <hardware>
-                <!-- By default, set up controllers for simulation. This won't work on real hardware -->
                 <plugin>mock_components/GenericSystem</plugin>
             </hardware>
-            <joint name="joint1">
+            <joint name="lift_joint">
                 <command_interface name="position"/>
                 <state_interface name="position">
-                  <param name="initial_value">${initial_positions['joint1']}</param>
+                    <param name="initial_value">${initial_positions['lift_joint']}</param>
                 </state_interface>
                 <state_interface name="velocity"/>
             </joint>
-            <joint name="joint2">
+            <joint name="head_joint1">
                 <command_interface name="position"/>
                 <state_interface name="position">
-                  <param name="initial_value">${initial_positions['joint2']}</param>
+                    <param name="initial_value">${initial_positions['head_joint1']}</param>
                 </state_interface>
                 <state_interface name="velocity"/>
             </joint>
-            <joint name="joint3">
+            <joint name="head_joint2">
                 <command_interface name="position"/>
                 <state_interface name="position">
-                  <param name="initial_value">${initial_positions['joint3']}</param>
+                    <param name="initial_value">${initial_positions['head_joint2']}</param>
                 </state_interface>
                 <state_interface name="velocity"/>
             </joint>
-            <joint name="joint4">
+            <joint name="virtual_gripper_joint">
                 <command_interface name="position"/>
                 <state_interface name="position">
-                  <param name="initial_value">${initial_positions['joint4']}</param>
-                </state_interface>
-                <state_interface name="velocity"/>
-            </joint>
-            <joint name="joint5">
-                <command_interface name="position"/>
-                <state_interface name="position">
-                  <param name="initial_value">${initial_positions['joint5']}</param>
-                </state_interface>
-                <state_interface name="velocity"/>
-            </joint>
-            <joint name="joint6">
-                <command_interface name="position"/>
-                <state_interface name="position">
-                  <param name="initial_value">${initial_positions['joint6']}</param>
-                </state_interface>
-                <state_interface name="velocity"/>
-            </joint>
-            <joint name="joint7">
-                <command_interface name="position"/>
-                <state_interface name="position">
-                  <param name="initial_value">${initial_positions['joint7']}</param>
-                </state_interface>
-                <state_interface name="velocity"/>
-            </joint>
-            <joint name="lift_joint">
-                <command_interface name="position"/>
-                <state_interface name="position">
-                  <param name="initial_value">${initial_positions['lift_joint']}</param>
+                    <param name="initial_value">${initial_positions['virtual_gripper_joint']}</param>
                 </state_interface>
                 <state_interface name="velocity"/>

File: src/kaair_moveit_config/config/kaair.urdf.xacro (robot description, xacro)
@@ -1,9 +1,38 @@
 <?xml version="1.0"?>
 <robot xmlns:xacro="http://www.ros.org/wiki/xacro" name="kaair">
-    <xacro:arg name="initial_positions_file" default="initial_positions.yaml" />
-    <!-- Import kaair urdf file -->
-    <xacro:include filename="$(find kaair_description)/urdf/robot.urdf.xacro" />
-    <!-- Import control_xacro -->
-    <xacro:include filename="kaair.ros2_control.xacro" />
-    <xacro:kaair_ros2_control name="FakeSystem" initial_positions_file="$(arg initial_positions_file)"/>
+    <!-- ── Arguments ──────────────────────────────────────────────────────────
+         use_fake_hardware      : true  → MoveIt fake mode (mock_components)
+                                  false → real hardware drivers
+         mode                   : robot | lift | arm | head | tool | slamtec
+         hw_spec_file           : robot hardware spec YAML (USB ports, limits …)
+         initial_positions_file : initial joint positions for FakeSystem
+    ──────────────────────────────────────────────────────────────────────── -->
+    <xacro:arg name="use_fake_hardware"      default="true"/>
+    <xacro:arg name="mode"                   default="robot"/>
+    <xacro:arg name="hw_spec_file"           default="$(find kaair_bringup)/config/robots/kaair_specs_01.yaml"/>
+    <xacro:arg name="initial_positions_file" default="$(find kaair_moveit_config)/config/initial_positions.yaml"/>
+    <!-- ── Robot description ──────────────────────────────────────────────────
+         Kinematics (links, joints, meshes) are always loaded from here.
+         ros2_control behaviour:
+           use_fake_hardware=false → per-subsystem real HW plugins are generated
+                                     (LiftHwInterface, HeadHwInterface,
+                                      UFRobotSystemHardware, ToolHwInterface)
+           use_fake_hardware=true  → kaair subsystem ros2_control blocks are
+                                     suppressed; arm gets UFRobotFakeSystemHardware
+                                     (joint1–7 only)
+    ──────────────────────────────────────────────────────────────────────── -->
+    <xacro:include filename="$(find kaair_description)/urdf/robot.urdf.xacro"/>
+    <!-- ── Fake hardware: single FakeSystem for KAAIR joints ─────────────────
+         Covers: lift_joint, head_joint1, head_joint2, virtual_gripper_joint
+         Initial positions loaded from initial_positions_file YAML.
+         arm joints (joint1–7) are NOT listed here — they are already provided
+         by UFRobotFakeSystemHardware in robot.urdf.xacro above. Listing them
+         in two ros2_control blocks would cause a ResourceManager conflict.
+    ──────────────────────────────────────────────────────────────────────── -->
+    <xacro:if value="$(arg use_fake_hardware)">
+        <xacro:include filename="$(find kaair_moveit_config)/config/kaair.ros2_control.xacro"/>
+        <xacro:kaair_ros2_control
+            name="FakeSystem"
+            initial_positions_file="$(arg initial_positions_file)"/>
+    </xacro:if>
 </robot>
