Commit message: xacro seperate control xacro

File: src/kaair_description/urdf/robot.urdf.xacro (robot description, xacro)
@@ -16,11 +16,24 @@
     <color rgba="0.8 0.8 0.8 1.0"/>
   </material>
-  <xacro:arg name="mode" default="robot"/>
-  <xacro:arg name="hw_spec_file" default="$(find kaair_bringup)/config/robots/kaair_specs_01.yaml"/>
-  <xacro:arg name="use_fake_hardware" default="false"/>
+  <xacro:arg name="mode"                  default="robot"/>
+  <xacro:arg name="hw_spec_file"          default="$(find kaair_bringup)/config/robots/kaair_specs_01.yaml"/>
+  <xacro:arg name="use_fake_hardware"     default="false"/>
+  <!--
+    include_ros2_control
+      true  (default) – 모든 <ros2_control> 블록 포함. 단일 CM 또는 하위 호환용.
+      false           – body 계열(lift/head/tool) <ros2_control> 블록 제외.
+                        RSP 전용 URDF로 사용할 때 지정한다.
+                        arm 섹션은 xacro:xarm_device 매크로가 <ros2_control> 블록을
+                        자동 생성하므로 완전 제외 불가. RSP 동작에는 영향 없음.
+                        2-CM 구조에서 arm CM은 arm_hw.urdf.xacro,
+                        body CM은 body_hw.urdf.xacro 를 각자의 robot_description 으로 사용한다.
+  -->
+  <xacro:arg name="include_ros2_control"  default="true"/>
   <xacro:property name="hw_specs" value="${xacro.load_yaml('$(arg hw_spec_file)')}"/>
+  <!-- ── Slamtec (mobile base) ────────────────────────────────────────── -->
   <xacro:if value="${'$(arg mode)' == 'robot' or '$(arg mode)' == 'slamtec'}">
     <xacro:include filename="$(find kaair_description)/urdf/slamtec/slamtec.urdf.xacro"/>
   </xacro:if>
+  <!-- ── Lift ─────────────────────────────────────────────────────────── -->
   <xacro:if value="${'$(arg mode)' == 'robot' or '$(arg mode)' == 'lift'}">
     <xacro:include filename="$(find kaair_description)/urdf/lift/lift.urdf.xacro"/>
@@ -30,12 +43,4 @@
       max_h="${hw_specs['lift']['max_h']}"
     />
-    <!-- real hw only: fake mode uses kaair_moveit_config/kaair.ros2_control.xacro FakeSystem -->
-    <xacro:unless value="$(arg use_fake_hardware)">
-      <xacro:lift_ros2_control
-        name="LiftHardware"
-        spec="${hw_specs['lift']}"
-        use_fake_hardware="false"
-      />
-    </xacro:unless>
     <xacro:if value="${'$(arg mode)' == 'robot'}">
       <joint name="lift_to_mobile_joint" type="fixed">
@@ -45,20 +50,23 @@
       </joint>
     </xacro:if>
+    <!-- ros2_control: include_ros2_control=true 이고 real HW 일 때만 삽입 -->
+    <xacro:if value="$(arg include_ros2_control)">
+      <xacro:unless value="$(arg use_fake_hardware)">
+        <xacro:lift_ros2_control
+          name="LiftHardware"
+          spec="${hw_specs['lift']}"
+          use_fake_hardware="false"
+        />
+      </xacro:unless>
+    </xacro:if>
   </xacro:if>
+  <!-- ── Head ─────────────────────────────────────────────────────────── -->
   <xacro:if value="${'$(arg mode)' == 'robot' or '$(arg mode)' == 'head'}">
     <xacro:include filename="$(find kaair_description)/urdf/head/head.urdf.xacro"/>
     <xacro:include filename="$(find kaair_description)/urdf/head/head.ros2_control.xacro"/>
     <xacro:include filename="$(find orbbec_description)/urdf/femto_bolt.urdf.xacro"/>
-    <!-- real hw only: fake mode uses kaair_moveit_config/kaair.ros2_control.xacro FakeSystem -->
-    <xacro:unless value="$(arg use_fake_hardware)">
-      <xacro:head_ros2_control
-        name="HeadHardware"
-        spec="${hw_specs['head']}"
-        use_fake_hardware="false"
-      />
-    </xacro:unless>
-  <xacro:femto_bolt prefix="femto" parent="head_camera_mount">
-    <origin xyz="0 0 0.01" rpy="0 0 0" />
-  </xacro:femto_bolt>
+    <xacro:femto_bolt prefix="femto" parent="head_camera_mount">
+      <origin xyz="0 0 0.01" rpy="0 0 0"/>
+    </xacro:femto_bolt>
     <xacro:if value="${'$(arg mode)' == 'robot'}">
       <joint name="lift_to_head_fix_joint" type="fixed">
@@ -68,5 +76,22 @@
       </joint>
     </xacro:if>
+    <!-- ros2_control: include_ros2_control=true 이고 real HW 일 때만 삽입 -->
+    <xacro:if value="$(arg include_ros2_control)">
+      <xacro:unless value="$(arg use_fake_hardware)">
+        <xacro:head_ros2_control
+          name="HeadHardware"
+          spec="${hw_specs['head']}"
+          use_fake_hardware="false"
+        />
+      </xacro:unless>
+    </xacro:if>
   </xacro:if>
+  <!-- ── Arm (xArm7) ──────────────────────────────────────────────────── -->
+  <!--
+    xacro:xarm_device 는 URDF 키네마틱과 <ros2_control> 블록을 함께 생성하는 매크로이므로
+    include_ros2_control=false 여도 <ros2_control> 블록이 포함된다.
+    RSP 는 이를 무시하므로 동작에 영향 없다.
+    2-CM 구조에서 실제 arm hardware 는 arm_hw.urdf.xacro 를 통해 arm CM 이 관리한다.
+  -->
   <xacro:if value="${'$(arg mode)' == 'robot' or '$(arg mode)' == 'arm'}">
     <xacro:unless value="${'$(arg mode)' == 'robot'}">
@@ -76,4 +101,9 @@
     <xacro:if value="$(arg use_fake_hardware)">
       <xacro:property name="arm_hw_plugin" value="uf_robot_hardware/UFRobotFakeSystemHardware"/>
+    </xacro:if>
+    <!-- include_ros2_control=false(RSP 전용)일 때는 GenericSystem 으로 대체하여
+         실제 HW 연결 시도 없이 키네마틱 구조만 사용한다. -->
+    <xacro:if value="${not '$(arg include_ros2_control)' == 'true'}">
+      <xacro:property name="arm_hw_plugin" value="mock_components/GenericSystem"/>
     </xacro:if>
     <xacro:include filename="$(find xarm_description)/urdf/xarm_device_macro.xacro"/>
@@ -91,4 +121,5 @@
     />
   </xacro:if>
+  <!-- ── Tool (gripper + D405) ────────────────────────────────────────── -->
   <xacro:if value="${'$(arg mode)' == 'robot' or '$(arg mode)' == 'tool'}">
     <xacro:include filename="$(find kaair_description)/urdf/tool/tool.urdf.xacro"/>
@@ -101,15 +132,17 @@
       </joint>
     </xacro:if>
-    <!-- real hw only: fake mode uses kaair_moveit_config/kaair.ros2_control.xacro FakeSystem -->
-    <xacro:unless value="$(arg use_fake_hardware)">
-      <xacro:tool_ros2_control
-        name="ToolHardware"
-        spec="${hw_specs['tool']}"
-        use_fake_hardware="false"
-      />
-    </xacro:unless>
+    <!-- ros2_control: include_ros2_control=true 이고 real HW 일 때만 삽입 -->
+    <xacro:if value="$(arg include_ros2_control)">
+      <xacro:unless value="$(arg use_fake_hardware)">
+        <xacro:tool_ros2_control
+          name="ToolHardware"
+          spec="${hw_specs['tool']}"
+          use_fake_hardware="false"
+        />
+      </xacro:unless>
+    </xacro:if>
     <xacro:arg name="use_nominal_extrinsics" default="false"/>
-    <xacro:arg name="add_plug" default="true"/>
-    <xacro:include filename="$(find realsense2_description)/urdf/_d405.urdf.xacro" />
+    <xacro:arg name="add_plug"               default="true"/>
+    <xacro:include filename="$(find realsense2_description)/urdf/_d405.urdf.xacro"/>
     <xacro:sensor_d405 parent="vision_frame_link" use_nominal_extrinsics="$(arg use_nominal_extrinsics)">
       <origin xyz="0.04428 0 0.02185" rpy="0 -1.5707963267948966 -3.1415926535897931"/>

File: src/kaair_moveit_config/config/kaair.urdf.xacro (robot description, xacro)
@@ -2,9 +2,10 @@
 <robot xmlns:xacro="http://www.ros.org/wiki/xacro" name="kaair">
     <!-- ── Arguments ──────────────────────────────────────────────────────────
-         use_fake_hardware      : true  → MoveIt fake mode (mock_components)
+         use_fake_hardware      : true  → MoveIt fake mode
                                   false → real hardware drivers
          mode                   : robot | lift | arm | head | tool | slamtec
-         hw_spec_file           : robot hardware spec YAML (USB ports, limits …)
-         initial_positions_file : initial joint positions for FakeSystem
+         hw_spec_file           : robot hardware spec YAML
+         initial_positions_file : (legacy) 하위 호환. 이 파일에서는 직접 사용하지 않음.
+                                  arm_hw / body_hw xacro 가 각자 사용한다.
     ──────────────────────────────────────────────────────────────────────── -->
     <xacro:arg name="use_fake_hardware"      default="true"/>
@@ -12,27 +13,16 @@
     <xacro:arg name="hw_spec_file"           default="$(find kaair_bringup)/config/robots/kaair_specs_01.yaml"/>
     <xacro:arg name="initial_positions_file" default="$(find kaair_moveit_config)/config/initial_positions.yaml"/>
-    <!-- ── Robot description ──────────────────────────────────────────────────
-         Kinematics (links, joints, meshes) are always loaded from here.
-         ros2_control behaviour:
-           use_fake_hardware=false → per-subsystem real HW plugins are generated
-                                     (LiftHwInterface, HeadHwInterface,
-                                      UFRobotSystemHardware, ToolHwInterface)
-           use_fake_hardware=true  → kaair subsystem ros2_control blocks are
-                                     suppressed; arm gets UFRobotFakeSystemHardware
-                                     (joint1–7 only)
+    <!-- ── include_ros2_control = false ──────────────────────────────────────
+         이 파일은 RSP / move_group 전용 URDF 이다.
+         ros2_control 블록은 2-CM 구조에서 각 CM 의 전용 xacro 가 담당한다.
+           arm CM  : arm_hw.urdf.xacro
+           body CM : body_hw.urdf.xacro
+         따라서 이 파일에서 ros2_control 을 포함하면 ResourceManager 충돌이 발생한다.
+         include_ros2_control:=false 를 강제하여 kinematics(링크/조인트)만 포함한다.
+         arm 섹션의 xacro:xarm_device 매크로는 ros2_control 블록을 자동 생성하지만,
+         include_ros2_control=false 일 때 mock_components/GenericSystem 으로 대체되므로
+         RSP 는 이를 무시하고 정상 동작한다.
     ──────────────────────────────────────────────────────────────────────── -->
+    <xacro:arg name="include_ros2_control" default="false"/>
     <xacro:include filename="$(find kaair_description)/urdf/robot.urdf.xacro"/>
-    <!-- ── Fake hardware: single FakeSystem for KAAIR joints ─────────────────
-         Covers: lift_joint, head_joint1, head_joint2, virtual_gripper_joint
-         Initial positions loaded from initial_positions_file YAML.
-         arm joints (joint1–7) are NOT listed here — they are already provided
-         by UFRobotFakeSystemHardware in robot.urdf.xacro above. Listing them
-         in two ros2_control blocks would cause a ResourceManager conflict.
-    ──────────────────────────────────────────────────────────────────────── -->
-    <xacro:if value="$(arg use_fake_hardware)">
-        <xacro:include filename="$(find kaair_moveit_config)/config/kaair.ros2_control.xacro"/>
-        <xacro:kaair_ros2_control
-            name="FakeSystem"
-            initial_positions_file="$(arg initial_positions_file)"/>
-    </xacro:if>
 </robot>
