Commit message: add 50mm tooltip

File: src/kaair_description/urdf/clober_robot.urdf.xacro (robot description, xacro)
@@ -15,4 +15,7 @@
   <material name="light_gray">
     <color rgba="0.8 0.8 0.8 1.0"/>
+  </material>
+  <material name="orange">
+    <color rgba="1.0 0.5 0.0 1.0"/>
   </material>
   <xacro:arg name="mode"                  default="robot"/>

File: src/kaair_description/urdf/robot.urdf.xacro (robot description, xacro)
@@ -15,4 +15,7 @@
   <material name="light_gray">
     <color rgba="0.8 0.8 0.8 1.0"/>
+  </material>
+  <material name="orange">
+    <color rgba="1.0 0.5 0.0 1.0"/>
   </material>
   <xacro:arg name="mode"                  default="robot"/>

File: src/kaair_description/urdf/tool/tool.urdf.xacro (robot description, xacro)
@@ -66,13 +66,13 @@
       <visual>
         <geometry>
-          <mesh filename="${mesh_path}tool/visual/left_finger.stl" scale="${m_to_mm}"/>
+          <mesh filename="${mesh_path}tool/visual/left_finger_tip_50mm.stl" scale="${m_to_mm}"/>
         </geometry>
         <origin xyz="0 0 0" rpy="0 0 0"/>
-        <material name="dark_gray"/>
+        <material name="orange"/>
       </visual>
       <!-- collision -->
       <collision>
         <geometry>
-          <mesh filename="${mesh_path}tool/visual/left_finger.stl" scale="${m_to_mm}"/>
+          <mesh filename="${mesh_path}tool/visual/left_finger_tip_50mm.stl" scale="${m_to_mm}"/>
         </geometry>
         <origin xyz="0 0 0" rpy="0 0 0"/>
@@ -83,13 +83,13 @@
       <visual>
         <geometry>
-          <mesh filename="${mesh_path}tool/visual/right_finger.stl" scale="${m_to_mm}"/>
+          <mesh filename="${mesh_path}tool/visual/right_finger_tip_50mm.stl" scale="${m_to_mm}"/>
         </geometry>
         <origin xyz="0 0 0" rpy="0 0 0"/>
-        <material name="dark_gray"/>
+        <material name="orange"/>
       </visual>
       <!-- collision -->
       <collision>
         <geometry>
-          <mesh filename="${mesh_path}tool/visual/right_finger.stl" scale="${m_to_mm}"/>
+          <mesh filename="${mesh_path}tool/visual/right_finger_tip_50mm.stl" scale="${m_to_mm}"/>
         </geometry>
         <origin xyz="0 0 0" rpy="0 0 0"/>
@@ -122,5 +122,5 @@
     </joint>
     <joint name="gripper_tcp_joint" type="fixed">
-      <origin xyz="0.0 0.0 0.241" rpy="0 0 0"/>
+      <origin xyz="0.0 0.0 0.191" rpy="0 0 0"/>
       <parent link="gripper_body_link"/>
       <child link="tool_tcp_link"/>
