Commit message: update clober base urdf

File: src/third_party/former_description/urdf/clober_500.urdf.xacro (robot description, xacro)
@@ -3,14 +3,10 @@
   <xacro:macro name="insert_robot" params="prefix">
   <xacro:include filename="$(find former_description)/urdf/common/tim571.urdf.xacro" />
-  <xacro:include filename="$(find realsense2_description)/urdf/_d435i.urdf.xacro" />
   <xacro:property name="PI" value="3.1415926535897931" />
-  <material name="black">
-    <color rgba="0.15 0.15 0.15 1.0" />
-  </material>
   <link name="base_footprint"/>
   <joint name="${prefix}base_link_fixed_joint" type="fixed">
     <parent link="${prefix}base_footprint"/>
     <child link="${prefix}base_link"/>
-    <origin xyz="0 0 0" rpy="0 0 0"/>
+    <origin xyz="0 0 0.02175" rpy="0 0 0"/>
   </joint>
   <link name="base_link">
@@ -22,11 +18,11 @@
     </visual>
     <collision>
-      <origin xyz="0 0 0" rpy="0 0 0" />
+      <origin xyz="0.0 0.0 0.142125" rpy="0 0 0"/>
       <geometry>
-        <mesh filename="package://former_description/meshes/clober_500.STL" />
+          <box size="0.5 0.5 0.32775"/>
       </geometry>
     </collision>
   </link>
-  <joint name="left_wheel_joint" type="continuous">
+  <joint name="left_wheel_joint" type="fixed">
     <parent link="base_link" />
     <child link="left_wheel_link" />
@@ -36,5 +32,5 @@
   <link name="left_wheel_link">
   </link>
-  <joint name="right_wheel_joint" type="continuous">
+  <joint name="right_wheel_joint" type="fixed">
     <parent link="base_link" />
     <child link="right_wheel_link" />
@@ -77,10 +73,4 @@
     <origin xyz="0.197 0 0.2885" rpy="${PI} 0 0" />
   </xacro:sensor_tim571>
-  <xacro:sensor_d435 parent="base_link" name="front_camera">
-    <origin xyz="0.225 0 0.135" rpy="0 0 0" />
-  </xacro:sensor_d435>
-  <xacro:sensor_d435 parent="base_link" name="rear_camera">
-    <origin xyz="-0.225 0 0.135" rpy="0 0 3.14" />
-  </xacro:sensor_d435>
   <!-- <ros2_control name="FormerSystem" type="system">
     <hardware>
