Commit message: gripper update

File: src/kaair_description/urdf/tool/tool.urdf.xacro (robot description, xacro)
@@ -83,4 +83,5 @@
       </collision>
     </link>
+    <link name="virtual_gripper_link"/>
     <joint name="hand_to_gripper_fix_joint" type="fixed">
       <origin xyz="0.0 0.0 0.0135" rpy="0 0 0"/>
@@ -93,20 +94,26 @@
       <child link="vision_frame_link"/>
     </joint>
-    <joint name="right_finger_tip_joint" type="prismatic">
-        <origin xyz="0.0 0.0035 0.15325" rpy="0 0 0"/>
-        <parent link="gripper_body_link"/>
-        <child link="right_finger_tip"/>
-        <axis xyz="0.0 1.0 0.0"/>
-        <limit upper="0.055" lower="0" effort="50"
-        velocity="0.005"/>
+    <joint name="virtual_gripper_joint" type="prismatic">
+      <origin xyz="0 0 0" rpy="0 0 0"/>
+      <parent link="hand_base_link"/>
+      <child link="virtual_gripper_link"/>
+      <axis xyz="0 1 0"/>
+      <limit upper="0.1" lower="0" effort="50" velocity="0.01"/>
     </joint>
-    <joint name="left_finger_tip_joint" type="prismatic">
-        <origin xyz="0.0 -0.0035 0.15325" rpy="0 0 0"/>
-        <parent link="gripper_body_link"/>
-        <child link="left_finger_tip"/>
-        <axis xyz="0.0 -1.0 0.0"/>
-        <limit upper="0.055" lower="0" effort="50"
-        velocity="0.005"/>
-        <mimic joint="right_finger_tip_joint" multiplier="1.0" offset="0"/>
-    </joint>
+  <joint name="right_finger_tip_joint" type="prismatic">
+    <origin xyz="0.0 0.0035 0.15325" rpy="0 0 0"/>
+    <parent link="gripper_body_link"/>
+    <child link="right_finger_tip"/>
+    <axis xyz="0.0 1.0 0.0"/>
+    <limit upper="0.05" lower="0" effort="50" velocity="0.005"/>
+    <mimic joint="virtual_gripper_joint" multiplier="0.5" offset="0"/>
+  </joint>
+  <joint name="left_finger_tip_joint" type="prismatic">
+    <origin xyz="0.0 -0.0035 0.15325" rpy="0 0 0"/>
+    <parent link="gripper_body_link"/>
+    <child link="left_finger_tip"/>
+    <axis xyz="0.0 -1.0 0.0"/>
+    <limit upper="0.05" lower="0" effort="50" velocity="0.005"/>
+    <mimic joint="virtual_gripper_joint" multiplier="0.5" offset="0"/>
+  </joint>
 </robot>

File: src/kaair_description/urdf/tool/tool_ros2_control.xacro (robot description, xacro)
@@ -13,10 +13,10 @@
           <param name="baud_rate">${spec['baud_rate']}</param>
         </xacro:unless> </hardware>
-      <joint name="right_finger_tip_joint">
+      <joint name="virtual_gripper_joint">
           <command_interface name="position">
           </command_interface>
           <command_interface name="velocity"/>
           <state_interface name="position">
-            <param name="initial_value">0.055</param>
+            <param name="initial_value">0.1</param>
           </state_interface>
           <state_interface name="velocity">

Commit message: testing fake moveit

File: src/kaair_description/urdf/tool/tool.urdf.xacro (robot description, xacro)
@@ -84,4 +84,5 @@
     </link>
     <link name="virtual_gripper_link"/>
+    <link name="tool_tcp_link"/>
     <joint name="hand_to_gripper_fix_joint" type="fixed">
       <origin xyz="0.0 0.0 0.0135" rpy="0 0 0"/>
@@ -100,4 +101,9 @@
       <axis xyz="0 1 0"/>
       <limit upper="0.1" lower="0" effort="50" velocity="0.01"/>
+    </joint>
+    <joint name="gripper_tcp_joint" type="fixed">
+      <origin xyz="0.0 0.0 0.241" rpy="0 0 0"/>
+      <parent link="gripper_body_link"/>
+      <child link="tool_tcp_link"/>
     </joint>
   <joint name="right_finger_tip_joint" type="prismatic">

Commit message: update examples

File: src/kaair_description/urdf/tool/tool.urdf.xacro (robot description, xacro)
@@ -105,5 +105,6 @@
       <child link="virtual_gripper_link"/>
       <axis xyz="0 1 0"/>
-      <limit upper="0.1" lower="0" effort="50" velocity="0.01"/>
+      <!-- 0.01 m/s 이면 전개 0.1 m 에 ~10 s → GripperAction stall_timeout 과 맞물려 실패하기 쉬움 -->
+      <limit upper="0.1" lower="0" effort="50" velocity="0.05"/>
     </joint>
     <joint name="gripper_tcp_joint" type="fixed">

Commit message: update srdf

File: src/kaair_description/urdf/tool/tool.urdf.xacro (robot description, xacro)
@@ -18,4 +18,12 @@
         </geometry>
         <origin xyz="0 0 0" rpy="0 0 0"/>
+      </collision>
+    </link>
+    <link name="tooltip_collision_link">
+      <collision>
+        <origin xyz="0.0 0.0 0.13" rpy="0 0 0"/>
+        <geometry>
+            <box size="0.028 0.170 0.13"/>
+        </geometry>
       </collision>
     </link>
@@ -95,4 +103,9 @@
       <child link="gripper_body_link"/>
     </joint>
+    <joint name="tooltip_dummpy_fix_joint" type="fixed">
+      <origin xyz="0.0 0.0 0.0" rpy="0 0 0"/>
+      <parent link="hand_base_link"/>
+      <child link="tooltip_collision_link"/>
+    </joint>
     <joint name="hand_to_vision_frame_fix_joint" type="fixed">
       <origin xyz="0.0 0.0 0.0" rpy="0 0 0"/>

Commit message: updated lift parallel

File: src/kaair_description/urdf/tool/tool.urdf.xacro (robot description, xacro)
@@ -24,5 +24,5 @@
         <origin xyz="0.0 0.0 0.13" rpy="0 0 0"/>
         <geometry>
-            <box size="0.028 0.170 0.13"/>
+            <box size="0.028 0.100 0.08"/>
         </geometry>
       </collision>
