Commit message: add camera calibration params

File: ros2/ros2_ws/src/kaair_description/urdf/clober_robot.urdf.xacro (robot description, xacro)
@@ -34,4 +34,11 @@
   <xacro:arg name="include_ros2_control"  default="true"/>
   <xacro:property name="hw_specs" value="${xacro.load_yaml('$(arg hw_spec_file)')}"/>
+  <!--
+    카메라 마운트 캘리브레이션 오프셋 [x, y, z, roll, pitch, yaw] (spec 파일, 키가 없으면 0).
+    D405 기본 자세가 pitch=-90° 이라 rpy를 성분별로 더하면 짐벌락으로 roll/yaw가 섞이므로,
+    부모 → *_calib_link(위치 + 보정 회전) → 카메라(기본 회전) 순으로 변환을 합성한다.
+  -->
+  <xacro:property name="femto_calib" value="${hw_specs.get('femto_calib', [0.0] * 6)}"/>
+  <xacro:property name="hand_calib"  value="${hw_specs.get('hand_calib', [0.0] * 6)}"/>
   <!-- ── Slamtec (mobile base) ────────────────────────────────────────── -->
   <xacro:if value="${'$(arg mode)' == 'robot' or '$(arg mode)' == 'clober'}">
@@ -70,6 +77,13 @@
     <xacro:include filename="$(find kaair_description)/urdf/head/head.ros2_control.xacro"/>
     <xacro:include filename="$(find orbbec_description)/urdf/femto_bolt.urdf.xacro"/>
-    <xacro:femto_bolt prefix="femto" parent="head_camera_mount">
-      <origin xyz="0 0 0.01" rpy="0 0 0"/>
+    <link name="femto_calib_link"/>
+    <joint name="femto_calib_joint" type="fixed">
+      <origin xyz="${0.0 + femto_calib[0]} ${0.0 + femto_calib[1]} ${0.01 + femto_calib[2]}"
+              rpy="${femto_calib[3]} ${femto_calib[4]} ${femto_calib[5]}"/>
+      <parent link="head_camera_mount"/>
+      <child link="femto_calib_link"/>
+    </joint>
+    <xacro:femto_bolt prefix="femto" parent="femto_calib_link">
+      <origin xyz="0 0 0" rpy="0 0 0"/>
     </xacro:femto_bolt>
     <xacro:if value="${'$(arg mode)' == 'robot'}">
@@ -148,6 +162,13 @@
     <xacro:arg name="add_plug"               default="true"/>
     <xacro:include filename="$(find realsense2_description)/urdf/_d405.urdf.xacro"/>
-    <xacro:sensor_d405 parent="vision_frame_link" use_nominal_extrinsics="$(arg use_nominal_extrinsics)">
-      <origin xyz="0.04428 0 0.02185" rpy="0 -1.5707963267948966 -3.1415926535897931"/>
+    <link name="hand_camera_calib_link"/>
+    <joint name="hand_camera_calib_joint" type="fixed">
+      <origin xyz="${0.04428 + hand_calib[0]} ${0.0 + hand_calib[1]} ${0.02185 + hand_calib[2]}"
+              rpy="${hand_calib[3]} ${hand_calib[4]} ${hand_calib[5]}"/>
+      <parent link="vision_frame_link"/>
+      <child link="hand_camera_calib_link"/>
+    </joint>
+    <xacro:sensor_d405 parent="hand_camera_calib_link" use_nominal_extrinsics="$(arg use_nominal_extrinsics)">
+      <origin xyz="0 0 0" rpy="0 -1.5707963267948966 -3.1415926535897931"/>
     </xacro:sensor_d405>
   </xacro:if>

File: ros2/ros2_ws/src/kaair_description/urdf/robot.urdf.xacro (robot description, xacro)
@@ -34,4 +34,11 @@
   <xacro:arg name="include_ros2_control"  default="true"/>
   <xacro:property name="hw_specs" value="${xacro.load_yaml('$(arg hw_spec_file)')}"/>
+  <!--
+    카메라 마운트 캘리브레이션 오프셋 [x, y, z, roll, pitch, yaw] (spec 파일, 키가 없으면 0).
+    D405 기본 자세가 pitch=-90° 이라 rpy를 성분별로 더하면 짐벌락으로 roll/yaw가 섞이므로,
+    부모 → *_calib_link(위치 + 보정 회전) → 카메라(기본 회전) 순으로 변환을 합성한다.
+  -->
+  <xacro:property name="femto_calib" value="${hw_specs.get('femto_calib', [0.0] * 6)}"/>
+  <xacro:property name="hand_calib"  value="${hw_specs.get('hand_calib', [0.0] * 6)}"/>
   <!-- ── Slamtec (mobile base) ────────────────────────────────────────── -->
   <xacro:if value="${'$(arg mode)' == 'robot' or '$(arg mode)' == 'slamtec'}">
@@ -69,6 +76,13 @@
     <xacro:include filename="$(find kaair_description)/urdf/head/head.ros2_control.xacro"/>
     <xacro:include filename="$(find orbbec_description)/urdf/femto_bolt.urdf.xacro"/>
-    <xacro:femto_bolt prefix="femto" parent="head_camera_mount">
-      <origin xyz="0 0 0.01" rpy="0 0 0"/>
+    <link name="femto_calib_link"/>
+    <joint name="femto_calib_joint" type="fixed">
+      <origin xyz="${0.0 + femto_calib[0]} ${0.0 + femto_calib[1]} ${0.01 + femto_calib[2]}"
+              rpy="${femto_calib[3]} ${femto_calib[4]} ${femto_calib[5]}"/>
+      <parent link="head_camera_mount"/>
+      <child link="femto_calib_link"/>
+    </joint>
+    <xacro:femto_bolt prefix="femto" parent="femto_calib_link">
+      <origin xyz="0 0 0" rpy="0 0 0"/>
     </xacro:femto_bolt>
     <xacro:if value="${'$(arg mode)' == 'robot'}">
@@ -147,6 +161,13 @@
     <xacro:arg name="add_plug"               default="true"/>
     <xacro:include filename="$(find realsense2_description)/urdf/_d405.urdf.xacro"/>
-    <xacro:sensor_d405 parent="vision_frame_link" use_nominal_extrinsics="$(arg use_nominal_extrinsics)">
-      <origin xyz="0.04428 0 0.02185" rpy="0 -1.5707963267948966 -3.1415926535897931"/>
+    <link name="hand_camera_calib_link"/>
+    <joint name="hand_camera_calib_joint" type="fixed">
+      <origin xyz="${0.04428 + hand_calib[0]} ${0.0 + hand_calib[1]} ${0.02185 + hand_calib[2]}"
+              rpy="${hand_calib[3]} ${hand_calib[4]} ${hand_calib[5]}"/>
+      <parent link="vision_frame_link"/>
+      <child link="hand_camera_calib_link"/>
+    </joint>
+    <xacro:sensor_d405 parent="hand_camera_calib_link" use_nominal_extrinsics="$(arg use_nominal_extrinsics)">
+      <origin xyz="0 0 0" rpy="0 -1.5707963267948966 -3.1415926535897931"/>
     </xacro:sensor_d405>
   </xacro:if>
